File: hardware/CC2640_interface.sch (EAGLE design)
At the start: 111 parts, among them IC1 MCP607-I/SN, IC2 TLC277IDR, Q1 FA-128, Q2 FC-12M, U1 MPU-9250, U2 INA321EA, U4 MCP73831, U6 XC6210, X1 USB-MICROB

Commit message: first rev done except antenna, antennas make a dude sad
Parts:
- removed L8: 22µH/±10%/1.7ohm/80mA(LB2012T220K/8030984), rcl:L-USL0805_5MIL_DWS
- removed PWR: GYX-SD-TC0805SURK(RED), DOUBLE-SIDE:LED0805DWS
- removed R29: 2k/1%, rcl:R-EU_R0603_5MIL_DWS
- removed SJ1: JUMPER-PAD-2-NC_BY_PASTEFULL-BOX-SILK, SparkFun-Passives:JUMPER-PAD-2-NC_BY_PASTEFULL-BOX-SILK
- added B130LAW: MBR0520LT, diode:MBR0520LT
- added C1: 1uF, SparkFun:CAP0402-CAP
- added DMP1045U: NX3008PBK, fets:NX3008PBK
- added Q3: MOSFET-NCHANNELSMD, fets:MOSFET-NCHANNELSMD
- added R25: (no value), passives:RESISTOR0603_RES
- added R28: 20k, SparkFun:RESISTOR0402-RES
- added SJ3: JUMPER-PAD-2-NC_BY_PASTEFULL-BOX-SILK, SparkFun-Passives:JUMPER-PAD-2-NC_BY_PASTEFULL-BOX-SILK
- R22, R23: value 10k/1% -> 20k/1%
- R4: value 10K -> 100k; device SparkFun-Resistors:10KOHM-1/10W-1%(0603)0603 -> SparkFun:RESISTOR0402-RES
Connections:
- removed net DIO_1: R4.1, U$1.DIO_1/SENSORCONTROL, U1.!CS
- removed net N$11: L8.1, PWR.A
- removed net N$12: DIG_POT.SHDWN_AL
- removed net N$15: PWR.C, R29.2
- removed net VDDIO: SJ1.2
- new net ANALOG_EN: Q3.G, R25.2, U$1.DIO_1/SENSORCONTROL
- new net LDO_IN: B130LAW.C, C1.1, C56.2, DMP1045U.D, U6.CE, U6.VIN
- new net SHDWN_AL: DIG_POT.SHDWN_AL, R28.1
- net +3V3: now also R28.2, SJ3.1, SJ3.2; no longer L8.2, R4.2, SJ1.1
- net 5VIN: now also B130LAW.A, DMP1045U.G, R4.1
- net DIO_10: now also U1.SCL/SCLK
- net DIO_11: now also U1.!CS; no longer U1.SCL/SCLK
- net DIO_12: no longer U1.SDA/SDI
- net DIO_9: now also U1.SDA/SDI
- net GND: now also C1.2, Q3.S, R25.1, R4.2
- net GNDA: now also Q3.D; no longer R29.1
- net VBATT: now also DMP1045U.S; no longer C56.2, U6.CE, U6.VIN
Other:
- note added: "put variable cap here"
- moved on the sheet: C29, L6
