File: hardware/CC2640_interface.sch (EAGLE design)
At the start: 114 parts, among them IC1 MCP607-I/SN, IC2 TLC277IDR, Q1 FA-128, Q2 FC-12M, Q3 MOSFET-NCHANNELSMD, U1 MPU-9250, U2 INA321EA, U4 MCP73831, U6 XC6210, X1 USB-MICROB

Commit message: we are shipping this
Parts:
- removed C2: 1.2 pF, rcl:C-EUC0402
- removed C3: 1 pF, rcl:C-EUC0402
- removed C4: 1.2pF, rcl:C-EUC0402
- removed L3, L4, L5: 2 nH, passives:INDUCTOR0603
- removed SJ3: JUMPER-PAD-2-NC_BY_PASTEFULL-BOX-SILK, SparkFun-Passives:JUMPER-PAD-2-NC_BY_PASTEFULL-BOX-SILK
- added JP1, JP2, JP3: (no value), pinhead:PINHD-1X2
- added SJ1, SJ2: JUMPER-PAD-2-NC_BY_PASTEFULL-BOX-SILK, SparkFun-Passives:JUMPER-PAD-2-NC_BY_PASTEFULL-BOX-SILK
- added U$2: 2450BM14G0011, chips:2450BM14G0011
- added U$3: ADG854, chips:ADG854
Connections:
- removed net N$4: C4.1, L3.2, L4.1
- removed net N$5: C3.1, L4.2, L5.1
- removed net RF_N: U$1.RF_N
- new net CH2_IN+: JP1.1, U$3.S1B
- new net CH2_IN-: JP1.2, U$3.S2B
- new net CHOSEN_POS: PGS2.1, R2.1, SJ2.1, U$3.D1
- new net CHOSE_NEG: PGS1.2, R3.1, SJ1.2, U$3.D2
- new net RF_NEG: U$1.RF_N, U$2.BAL_N
- new net SWITCH: U$1.DIO_3/SC/HD, U$3.IN1, U$3.IND2
- net +3V3: now also U$3.VDD; no longer SJ3.1, SJ3.2
- net CH1_IN+: now also SJ2.2, U$3.S1A; no longer PGS2.1, R2.1
- net CH1_IN-: now also SJ1.1, U$3.S2A; no longer PGS1.2, R3.1
- net GND: now also U$2.GND, U$2.GND1, U$3.GND; no longer C2.2, C3.2, C4.2
- net JTAG_TCKC: now also JP2.1
- net JTAG_TDI: now also JP3.1
- net JTAG_TDO: now also JP3.2
- net JTAG_TSMC: now also JP2.2
- net N$7: now also U$2.ANT; no longer L5.2
- net RF_P: now also U$2.BAL_P; no longer C2.1, L3.1
Other:
- note added: "3 switches"
- note added: "programming pins here"
- moved on the sheet: SV1
